Commit message: zed mesh is added.

File: aion_descriptions/aion_r1_description/urdf/r1_sim.urdf.xacro (robot description, xacro)
@@ -196,5 +196,5 @@
       <origin xyz="0 0 0" rpy="0 0 0"/>
       <geometry>
-        <mesh filename="package://zed_wrapper/urdf/models/ZED.stl" />
+        <mesh filename="package://aion_r1_description/meshes/ZED.stl" />
       </geometry>
       <material name="light_grey">
@@ -217,5 +217,5 @@
       <collision>
       <geometry>
-        <mesh filename="package://zed_wrapper/urdf/models/ZED.stl" />
+        <mesh filename="package://aion_r1_description/meshes/ZED.stl" />
       </geometry>
     </collision>

Commit message: revised at outdoor experiment. 10/6

File: aion_descriptions/aion_r1_description/urdf/r1_sim.urdf.xacro (robot description, xacro)
@@ -91,5 +91,5 @@
   </xacro:macro>
   <!-- Defining model links. -->
-	<link name="odom" />
+	<link name="UGV/odom" />
   <link
     name="base_link">
@@ -251,5 +251,5 @@
     name="fixed_base_joint"
     type="fixed">
-    <parent link="odom" />
+    <parent link="UGV/odom" />
     <child link="base_link" />
   </joint>

Commit message: r1_description is revised

File: aion_descriptions/aion_r1_description/urdf/r1_sim.urdf.xacro (robot description, xacro)
@@ -91,5 +91,5 @@
   </xacro:macro>
   <!-- Defining model links. -->
-	<link name="UGV/odom" />
+	<link name="odom" />
   <link
     name="base_link">
@@ -251,5 +251,5 @@
     name="fixed_base_joint"
     type="fixed">
-    <parent link="UGV/odom" />
+    <parent link="odom" />
     <child link="base_link" />
   </joint>

Commit message: tf issue V01.

File: aion_descriptions/aion_r1_description/urdf/r1_sim.urdf.xacro (robot description, xacro)
@@ -92,5 +92,5 @@
   <!-- Defining model links. -->
 	<link name="UGV/odom" />
-  <link
+ <link
     name="base_link">
     <inertial>
