Commit message: zed is removed. V02

File: aion_descriptions/aion_r1_description/urdf/r1_without_ZED.urdf.xacro (robot description, xacro)
@@ -91,5 +91,5 @@
   </xacro:macro>
   <!-- Defining model links. -->
-	<link name="odom" />
+	<link name="UGV/odom" />
   <link
     name="base_link">
@@ -196,5 +196,5 @@
     name="fixed_base_joint"
     type="fixed">
-    <parent link="odom" />
+    <parent link="UGV/odom" />
     <child link="base_link" />
   </joint>
